File: Eagle/Downconverter.sch (EAGLE design)
At the start: 26 parts, among them J2 3.5HEADPHONEJACK, J5 U.FL_CONN, J6 U.FL_CONN, U1 5V_REG, U2 MIXER, U3 DUAL_OP_AMP_LMV822, U4 DIGITAL_POTDIGITAL_POT

Commit message: Done routing.
Connections:
- net 5V: no longer J3.2
- net 9V: now also J3.2
Other:
- note added: "9V"
Changed lines of the file:
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@@
 <part name="GND3" library="SparkFun-PowerSymbols" library_urn="urn:adsk.eagle:library:530" deviceset="GND" device=""/>
 <part name="J3" library="SparkFun-Connectors" library_urn="urn:adsk.eagle:library:513" deviceset="CONN_02" device="" package3d_urn="urn:adsk.eagle:package:38039/1"/>
-<part name="SUPPLY3" library="SparkFun-PowerSymbols" library_urn="urn:adsk.eagle:library:530" deviceset="5V" device=""/>
 <part name="GND2" library="SparkFun-PowerSymbols" library_urn="urn:adsk.eagle:library:530" deviceset="GND" device=""/>
 <part name="U2" library="764Library" deviceset="MIXER" device=""/>
@@
 <part name="J8" library="SparkFun-Connectors" library_urn="urn:adsk.eagle:library:513" deviceset="CONN_02" device="" package3d_urn="urn:adsk.eagle:package:38039/1"/>
 <part name="GND15" library="SparkFun-PowerSymbols" library_urn="urn:adsk.eagle:library:530" deviceset="GND" device=""/>
+<part name="9V1" library="SparkFun-PowerSymbols" library_urn="urn:adsk.eagle:library:530" deviceset="V_BATT" device=""/>
 </parts>
 <sheets>
@@
 <wire x1="170.18" y1="10.16" x2="132.08" y2="10.16" width="0.1524" layer="97" style="shortdash"/>
 <wire x1="132.08" y1="10.16" x2="132.08" y2="50.8" width="0.1524" layer="97" style="shortdash"/>
+<text x="10.16" y="116.84" size="1.778" layer="97">9V</text>
 </plain>
 <instances>
@@
 <attribute name="NAME" x="81.28" y="107.188" size="1.778" layer="95" font="vector"/>
 </instance>
-<instance part="SUPPLY3" gate="G$1" x="91.44" y="114.3" smashed="yes">
-<attribute name="VALUE" x="91.44" y="117.094" size="1.778" layer="96" align="bottom-center"/>
-</instance>
 <instance part="GND2" gate="1" x="91.44" y="91.44" smashed="yes">
 <attribute name="VALUE" x="91.44" y="91.186" size="1.778" layer="96" align="top-center"/>
@@
 <instance part="GND15" gate="1" x="281.94" y="-7.62" smashed="yes">
 <attribute name="VALUE" x="281.94" y="-7.874" size="1.778" layer="96" align="top-center"/>
+</instance>
+<instance part="9V1" gate="G$1" x="91.44" y="114.3" smashed="yes">
+<attribute name="VALUE" x="91.44" y="117.094" size="1.778" layer="96" align="bottom-center"/>
 </instance>
 </instances>
@@
 <wire x1="20.32" y1="101.6" x2="20.32" y2="106.68" width="0.1524" layer="91"/>
 <pinref part="9V" gate="G$1" pin="V_BATT"/>
-<label x="20.32" y="109.22" size="1.778" layer="95"/>
 <wire x1="20.32" y1="106.68" x2="20.32" y2="114.3" width="0.1524" layer="91"/>
 <junction x="20.32" y="106.68"/>
@@
 <junction x="30.48" y="106.68"/>
 </segment>
+<segment>
+<pinref part="J3" gate="G$1" pin="2"/>
+<wire x1="91.44" y1="104.14" x2="91.44" y2="114.3" width="0.1524" layer="91"/>
+<pinref part="9V1" gate="G$1" pin="V_BATT"/>
+</segment>
 </net>
 <net name="N$1" class="0">
@@
 </segment>
 <segment>
-<pinref part="J3" gate="G$1" pin="2"/>
-<wire x1="91.44" y1="104.14" x2="91.44" y2="114.3" width="0.1524" layer="91"/>
-<pinref part="SUPPLY3" gate="G$1" pin="5V"/>
-</segment>
-<segment>

Commit message: Complete, just need to add taps
Other:
- note added: "-56 dBm 2.5E-9W 0.000248 V"
- note added: "Low Pass Filter fc = 5k Gain = R5/R4 = 100"
- note added: "MCA1-85L+ ASSUME CONVERSION LOSS 6dBm"
- note removed: "-56 dBm 2.5E-9 0.000248 V"
- note removed: "LPF fc = 5k Gain = R5/R4 = 100"
- note removed: "MCA1-85L+ ASSUME INSERTION LOSS 6dBm"
Changed lines of the file:
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@@
 <text x="139.7" y="134.62" size="2.54" layer="97">Downconverter/Preamp - Miranda Dodson</text>
 <text x="86.36" y="83.82" size="1.778" layer="97" align="top-left">To TX/RX</text>
-<text x="142.24" y="-40.64" size="1.778" layer="97">LPF fc = 5k
+<text x="142.24" y="-43.18" size="1.778" layer="97">Low Pass Filter
+fc = 5k
 Gain = R5/R4 = 100</text>
 <text x="198.12" y="-17.78" size="1.778" layer="97" align="bottom-right">N/C</text>
@@
 <text x="177.8" y="53.34" size="1.778" layer="97">LM821 OP AMP</text>
 <text x="76.2" y="-10.16" size="1.778" layer="97">MCA1-85L+
-ASSUME INSERTION
+ASSUME CONVERSION
 LOSS 6dBm</text>
 <text x="68.58" y="55.88" size="1.778" layer="97">-50 dBm
@@
 0.624V</text>
 <text x="96.52" y="43.18" size="1.778" layer="97">-56 dBm
-2.5E-9
+2.5E-9W
 0.000248 V</text>
 <text x="66.04" y="124.46" size="1.778" layer="97">Supply Voltage Conversion</text>
@@
 <wire x1="132.08" y1="10.16" x2="132.08" y2="50.8" width="0.1524" layer="97" style="shortdash"/>
 <text x="10.16" y="116.84" size="1.778" layer="97">9V</text>
+<wire x1="114.3" y1="-12.7" x2="180.34" y2="-12.7" width="0.1524" layer="97" style="shortdash"/>
+<wire x1="114.3" y1="-33.02" x2="180.34" y2="-33.02" width="0.1524" layer="97" style="shortdash"/>
+<wire x1="114.3" y1="-12.7" x2="114.3" y2="-33.02" width="0.1524" layer="97" style="shortdash"/>
+<wire x1="180.34" y1="-12.7" x2="180.34" y2="-33.02" width="0.1524" layer="97" style="shortdash"/>
 </plain>
 <instances>
