File: Eagle/Downconverter.brd (EAGLE design)
At the start: 40 x 40 mm, 26 parts, among them J2 3.5HEADPHONEJACK, J5 U.FL_CONN, J6 U.FL_CONN, U1 5V_REG, U2 MIXER, U3 DUAL_OP_AMP_LMV822, U4 DIGITAL_POTDIGITAL_POT

Commit message: Done routing.
Parts:
- moved J3 1.53 mm to (4.70, 36.1), turned to 180 degrees
- moved C4 0.64 mm to (22.9, 13.0)
- moved J7 0.63 mm to (37.5, 2.54)
- moved R4 0.32 mm to (15.9, 3.17)
Connections:
- net 5V: no longer J3.2
- net 9V: now also J3.2
Routing:
- net 9V: track 8.82 -> 21.1 mm
- net N$13: track 14.4 -> 23.7 mm, vias 2 -> 0
- net GND: track 37.1 -> 45.4 mm, vias 22 -> 23
- net N$12: track 39.2 -> 36.7 mm
- net 5V: track 51.4 -> 49.4 mm
- net SDI: track 11.7 -> 10.3 mm
- net SCK: track 11.0 -> 9.66 mm
- net SHDN: track 11.5 -> 10.4 mm
- net 5.8GHZ: track 1.97 -> 2.92 mm
- net SDO: track 9.98 -> 9.15 mm
- net CS: track 9.91 -> 9.09 mm
- net RAW_RF: track 1.97 -> 2.77 mm

Commit message: Complete, just need to add taps
Parts:
- moved J2 0.52 mm to (28.7, 29.1)
Routing:
- net N$12: track 36.7 -> 38.1 mm
- net RDR_OUT: track 37.4 -> 38.5 mm
- net GND: track 45.4 -> 44.4 mm
Other:
- board text added: "+"
- board text added: "3.3 V"
- board text added: "3.3V FROM TEENSY 3.2"
- board text added: "5.8 GHz REFERENCE"
- board text added: "5V"
- board text added: "5V to Teensy 3.2"
- board text added: "9V BATTERY"
- board text added: "9V BATTERY TO TX/RX"
- board text added: "CS"
- board text added: "ECE 764 K.I.S.S. Radar DOWNCONVERTER/PREAMP MIRANDA DODSON REV 0"
- board text added: "GND"
- board text added: "RAW RF SIGNAL"
- board text added: "RDR_OUT"
- board text added: "SCK"
- board text added: "SDI"
- board text added: "SDO"
- board text added: "SHDN"
- board text added: "TO TEENSY 3.2"

Commit message: Finished Rev 0 for Downconverter
Routing:
- net 5V: track 49.4 -> 51.8 mm, vias 0 -> 1
Other:
- board text added: "TP1"
- board text added: "To Teensy 3.2"
- board text removed: "5V to Teensy 3.2"
Changed lines of the file:
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@@
 <text x="15.494" y="38.735" size="0.4064" layer="21">TO TEENSY 3.2</text>
 <text x="26.035" y="5.08" size="0.4064" layer="21" rot="R180">3.3V FROM TEENSY 3.2</text>
-<text x="21.463" y="2.667" size="0.4064" layer="21" rot="R90">GND</text>
-<text x="27.686" y="2.667" size="0.4064" layer="21" rot="R90">3.3 V</text>
-<text x="39.243" y="20.574" size="0.4064" layer="21" rot="R180">5V to Teensy 3.2</text>
+<text x="27.813" y="2.667" size="0.4064" layer="21" rot="R90">GND</text>
+<text x="21.59" y="2.54" size="0.4064" layer="21" rot="R90">3.3 V</text>
+<text x="39.243" y="20.574" size="0.4064" layer="21" rot="R180">To Teensy 3.2</text>
 <text x="35.306" y="17.653" size="0.4064" layer="21">5V</text>
 <text x="35.052" y="15.24" size="0.4064" layer="21">CS</text>
@@
 <text x="5.969" y="17.78" size="0.4064" layer="21" rot="R180">5.8 GHz REFERENCE</text>
 <text x="18.161" y="11.049" size="0.4064" layer="21" rot="R180">RAW RF SIGNAL</text>
-<dimension x1="0" y1="0" x2="40" y2="0" x3="20" y3="-8.128" textsize="0.4064" layer="150"/>
-<dimension x1="40" y1="0" x2="40" y2="40" x3="48.133" y3="20" textsize="0.4064" layer="150"/>
+<dimension x1="0" y1="0" x2="40" y2="0" x3="20" y3="-8.128" textsize="0.4064" layer="150" visible="yes"/>
+<dimension x1="40" y1="0" x2="40" y2="40" x3="48.133" y3="20" textsize="0.4064" layer="150" visible="yes"/>
+<text x="17.272" y="30.48" size="0.4064" layer="21" rot="R180">TP1</text>
 </plain>
 <attributes>
@@
 <wire x1="12.8025" y1="33.87" x2="14.605" y2="32.0675" width="0.6096" layer="1"/>
 <wire x1="25.9588" y1="19.05" x2="24.4475" y2="19.05" width="0.6096" layer="1"/>
-<wire x1="24.4475" y1="19.05" x2="15.875" y2="27.6225" width="0.6096" layer="1"/>
+<wire x1="24.4475" y1="19.05" x2="16.79575" y2="26.70175" width="0.6096" layer="1"/>
+<wire x1="16.79575" y1="26.70175" x2="15.875" y2="27.6225" width="0.6096" layer="1"/>
 <wire x1="26.035" y1="20.74" x2="25.9588" y2="20.6638" width="0.6096" layer="1"/>
 <wire x1="25.9588" y1="20.6638" x2="25.9588" y2="19.05" width="0.6096" layer="1"/>
@@
 <wire x1="15.875" y1="27.6225" x2="14.8725" y2="27.6225" width="0.6096" layer="1"/>
 <wire x1="14.8725" y1="27.6225" x2="14.555" y2="27.305" width="0.6096" layer="1"/>
+<via x="16.764" y="29.083" extent="1-16" drill="1.016" shape="square"/>
+<wire x1="16.79575" y1="26.70175" x2="16.79575" y2="29.05125" width="0.635" layer="1"/>
+<wire x1="16.79575" y1="29.05125" x2="16.764" y2="29.083" width="0.4064" layer="1"/>
 </signal>
 <signal name="RAW_RF">
