File: Eagle/DSP.sch (EAGLE design)
At the start: 23 parts

Commit message: finished DSP layout!
Connections:
- net +3V3: now also J3.5; no longer J3.3
- net GND: now also C6.2
- net MISO: now also J3.1; no longer J3.2
- net MOSI: now also J3.2; no longer J3.1
- net SCLK: now also J3.3; no longer J3.5
Changed lines of the file:
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@@
 <instance part="SUPPLY4" gate="GND" x="40.64" y="71.12"/>
 <instance part="SUPPLY5" gate="GND" x="86.36" y="71.12"/>
-<instance part="+3V2" gate="G$1" x="213.36" y="78.74"/>
+<instance part="+3V2" gate="G$1" x="213.36" y="81.28"/>
 <instance part="C1" gate="G$1" x="198.12" y="68.58"/>
 <instance part="SUPPLY2" gate="GND" x="198.12" y="58.42"/>
@@
 <instance part="+3V4" gate="G$1" x="101.6" y="147.32"/>
 <instance part="SUPPLY8" gate="GND" x="101.6" y="106.68"/>
-<instance part="+3V5" gate="G$1" x="60.96" y="124.46"/>
-<instance part="SUPPLY9" gate="GND" x="50.8" y="106.68"/>
+<instance part="+3V5" gate="G$1" x="50.8" y="139.7"/>
+<instance part="SUPPLY9" gate="GND" x="50.8" y="104.14"/>
 <instance part="J4" gate="G$1" x="-12.7" y="139.7" rot="MR180"/>
 <instance part="SUPPLY10" gate="GND" x="0" y="129.54"/>
@@
 <wire x1="30.48" y1="116.84" x2="50.8" y2="116.84" width="0.1524" layer="91"/>
 <pinref part="SUPPLY9" gate="GND" pin="GND"/>
-<wire x1="50.8" y1="116.84" x2="50.8" y2="109.22" width="0.1524" layer="91"/>
+<wire x1="50.8" y1="116.84" x2="50.8" y2="106.68" width="0.1524" layer="91"/>
 <pinref part="J3" gate="G$1" pin="4"/>
 </segment>
@@
 </segment>
 <segment>
+<pinref part="C6" gate="G$1" pin="2"/>
 <pinref part="SUPPLY14" gate="GND" pin="GND"/>
 <wire x1="208.28" y1="60.96" x2="208.28" y2="63.5" width="0.1524" layer="91"/>
@@
 </segment>
 <segment>
-<pinref part="+3V5" gate="G$1" pin="+3V3"/>
-<wire x1="60.96" y1="121.92" x2="60.96" y2="114.3" width="0.1524" layer="91"/>
-<wire x1="60.96" y1="114.3" x2="30.48" y2="114.3" width="0.1524" layer="91"/>
-<pinref part="J3" gate="G$1" pin="3"/>
-</segment>
-<segment>
 <pinref part="J4" gate="G$1" pin="1"/>
 <pinref part="+3V6" gate="G$1" pin="+3V3"/>
@@
 <segment>
 <pinref part="+3V2" gate="G$1" pin="+3V3"/>
-<wire x1="213.36" y1="76.2" x2="213.36" y2="73.66" width="0.1524" layer="91"/>
+<wire x1="213.36" y1="78.74" x2="213.36" y2="73.66" width="0.1524" layer="91"/>
 <wire x1="213.36" y1="73.66" x2="208.28" y2="73.66" width="0.1524" layer="91"/>
 <pinref part="C1" gate="G$1" pin="1"/>
@@
 <junction x="208.28" y="73.66"/>
 </segment>
+<segment>
+<pinref part="J3" gate="G$1" pin="5"/>
+<wire x1="30.48" y1="119.38" x2="50.8" y2="119.38" width="0.1524" layer="91"/>
+<pinref part="+3V5" gate="G$1" pin="+3V3"/>
+<wire x1="50.8" y1="119.38" x2="50.8" y2="137.16" width="0.1524" layer="91"/>
+</segment>
 </net>
 <net name="N$1" class="0">
@@
 </segment>
 <segment>
-<wire x1="33.02" y1="109.22" x2="30.48" y2="109.22" width="0.1524" layer="91"/>
-<label x="33.02" y="109.22" size="1.778" layer="95"/>
-<pinref part="J3" gate="G$1" pin="1"/>
+<pinref part="J3" gate="G$1" pin="2"/>
+<wire x1="33.02" y1="111.76" x2="30.48" y2="111.76" width="0.1524" layer="91"/>
+<label x="33.02" y="111.76" size="1.778" layer="95"/>
 </segment>
 </net>
@@
 </segment>
 <segment>
-<wire x1="33.02" y1="111.76" x2="30.48" y2="111.76" width="0.1524" layer="91"/>
-<label x="33.02" y="111.76" size="1.778" layer="95"/>
-<pinref part="J3" gate="G$1" pin="2"/>
+<pinref part="J3" gate="G$1" pin="1"/>
+<wire x1="33.02" y1="109.22" x2="30.48" y2="109.22" width="0.1524" layer="91"/>
+<label x="33.02" y="109.22" size="1.778" layer="95"/>
 </segment>
 </net>
@@
 </segment>
 <segment>
-<wire x1="30.48" y1="119.38" x2="33.02" y2="119.38" width="0.1524" layer="91"/>
-<label x="33.02" y="119.38" size="1.778" layer="95"/>
-<pinref part="J3" gate="G$1" pin="5"/>
-</segment>
-</net>
+<pinref part="J3" gate="G$1" pin="3"/>
+<wire x1="33.02" y1="114.3" x2="30.48" y2="114.3" width="0.1524" layer="91"/>
+<label x="33.02" y="114.3" size="1.778" layer="95"/>
+</segment>
+</net>

Commit message: updates to dsp layout
Other:
- note added: "128x64 LCD Display"
- note added: "ADC Input Offset"
- note added: "Microcontroller and LED Array"
- note added: "Mode and Channel Switches"
- note added: "Off-Board Connectors"
- moved on the sheet: C1, C2, C3, C4, C5, C6, D1, J1, J2, J3, J4, J5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

Commit message: w00f
Parts:
- added C7: 0.22uF, kiss_z:C0603
- added R8: 1K, kiss_z:R0603
Connections:
- new net N$24: C7.1, R2.1, R8.2
- net +3V3: now also R8.1; no longer R2.1
- net GND: now also C7.2
Other:
- moved on the sheet: C2, R2, R3
Changed lines of the file:
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@@
 <part name="C6" library="kiss_z" deviceset="C0603" device="" value="0.1uF"/>
 <part name="SUPPLY14" library="supply2" library_urn="urn:adsk.eagle:library:372" deviceset="GND" device=""/>
+<part name="C7" library="kiss_z" deviceset="C0603" device="" value="0.22uF"/>
+<part name="SUPPLY15" library="supply2" library_urn="urn:adsk.eagle:library:372" deviceset="GND" device=""/>
+<part name="R8" library="kiss_z" deviceset="R0603" device="" value="1K"/>
 </parts>
 <sheets>
@@
 <instance part="J2" gate="G$1" x="17.78" y="167.64" rot="MR180"/>
 <instance part="SUPPLY7" gate="GND" x="30.48" y="157.48"/>
-<instance part="R2" gate="G$1" x="165.1" y="185.42" rot="R270"/>
-<instance part="R3" gate="G$1" x="165.1" y="170.18" rot="R270"/>
-<instance part="C2" gate="G$1" x="152.4" y="177.8" rot="R90"/>
-<instance part="+3V4" gate="G$1" x="165.1" y="198.12"/>
-<instance part="SUPPLY8" gate="GND" x="165.1" y="157.48"/>
+<instance part="R2" gate="G$1" x="167.64" y="162.56" rot="R270"/>
+<instance part="R3" gate="G$1" x="167.64" y="147.32" rot="R270"/>
+<instance part="C2" gate="G$1" x="154.94" y="154.94" rot="R90"/>
+<instance part="+3V4" gate="G$1" x="152.4" y="193.04"/>
+<instance part="SUPPLY8" gate="GND" x="167.64" y="134.62"/>
 <instance part="+3V5" gate="G$1" x="114.3" y="190.5"/>
 <instance part="SUPPLY9" gate="GND" x="114.3" y="154.94"/>
@@
 <instance part="C6" gate="G$1" x="266.7" y="86.36"/>
 <instance part="SUPPLY14" gate="GND" x="266.7" y="76.2"/>
+<instance part="C7" gate="G$1" x="182.88" y="180.34"/>
+<instance part="SUPPLY15" gate="GND" x="182.88" y="170.18"/>
+<instance part="R8" gate="G$1" x="160.02" y="185.42"/>
 </instances>
 <busses>
@@
 <pinref part="R3" gate="G$1" pin="2"/>
 <pinref part="SUPPLY8" gate="GND" pin="GND"/>
-<wire x1="165.1" y1="165.1" x2="165.1" y2="160.02" width="0.1524" layer="91"/>
+<wire x1="167.64" y1="142.24" x2="167.64" y2="137.16" width="0.1524" layer="91"/>
 </segment>
 <segment>
@@
 <pinref part="SUPPLY14" gate="GND" pin="GND"/>
 <wire x1="266.7" y1="78.74" x2="266.7" y2="81.28" width="0.1524" layer="91"/>
+</segment>
+<segment>
+<pinref part="C7" gate="G$1" pin="2"/>
+<pinref part="SUPPLY15" gate="GND" pin="GND"/>
+<wire x1="182.88" y1="172.72" x2="182.88" y2="175.26" width="0.1524" layer="91"/>
 </segment>
 </net>
@@
 <pinref part="+3V3" gate="G$1" pin="+3V3"/>
 <wire x1="35.56" y1="66.04" x2="35.56" y2="71.12" width="0.1524" layer="91"/>
-</segment>
-<segment>
-<pinref part="+3V4" gate="G$1" pin="+3V3"/>
-<pinref part="R2" gate="G$1" pin="1"/>
-<wire x1="165.1" y1="195.58" x2="165.1" y2="190.5" width="0.1524" layer="91"/>
 </segment>
 <segment>
@@
 <wire x1="114.3" y1="170.18" x2="114.3" y2="187.96" width="0.1524" layer="91"/>
 </segment>
+<segment>
+<pinref part="R8" gate="G$1" pin="1"/>
+<wire x1="154.94" y1="185.42" x2="152.4" y2="185.42" width="0.1524" layer="91"/>
+<pinref part="+3V4" gate="G$1" pin="+3V3"/>
+<wire x1="152.4" y1="185.42" x2="152.4" y2="190.5" width="0.1524" layer="91"/>
+</segment>
 </net>
 <net name="N$1" class="0">
@@
 <pinref part="R2" gate="G$1" pin="2"/>
 <pinref part="R3" gate="G$1" pin="1"/>
-<wire x1="165.1" y1="180.34" x2="165.1" y2="177.8" width="0.1524" layer="91"/>
-<wire x1="165.1" y1="177.8" x2="165.1" y2="175.26" width="0.1524" layer="91"/>
-<wire x1="165.1" y1="177.8" x2="157.48" y2="177.8" width="0.1524" layer="91"/>
-<junction x="165.1" y="177.8"/>
+<wire x1="167.64" y1="157.48" x2="167.64" y2="154.94" width="0.1524" layer="91"/>
+<wire x1="167.64" y1="154.94" x2="167.64" y2="152.4" width="0.1524" layer="91"/>
+<wire x1="167.64" y1="154.94" x2="160.02" y2="154.94" width="0.1524" layer="91"/>
+<junction x="167.64" y="154.94"/>
 <pinref part="C2" gate="G$1" pin="2"/>
-<wire x1="165.1" y1="177.8" x2="172.72" y2="177.8" width="0.1524" layer="91"/>
-<label x="172.72" y="177.8" size="1.778" layer="95"/>
+<wire x1="167.64" y1="154.94" x2="175.26" y2="154.94" width="0.1524" layer="91"/>
+<label x="175.26" y="154.94" size="1.778" layer="95"/>
 </segment>
 <segment>
@@
 <segment>
 <pinref part="C2" gate="G$1" pin="1"/>
-<wire x1="144.78" y1="177.8" x2="149.86" y2="177.8" width="0.1524" layer="91"/>
-<label x="144.78" y="177.8" size="1.778" layer="95" rot="MR0"/>
+<wire x1="147.32" y1="154.94" x2="152.4" y2="154.94" width="0.1524" layer="91"/>
+<label x="147.32" y="154.94" size="1.778" layer="95" rot="MR0"/>
 </segment>
 <segment>
@@
 </segment>
 </net>
+<net name="N$24" class="0">
+<segment>
+<wire x1="167.64" y1="185.42" x2="182.88" y2="185.42" width="0.1524" layer="91"/>
+<pinref part="C7" gate="G$1" pin="1"/>
+<wire x1="182.88" y1="185.42" x2="182.88" y2="182.88" width="0.1524" layer="91"/>
+<pinref part="R2" gate="G$1" pin="1"/>
+<wire x1="167.64" y1="185.42" x2="167.64" y2="167.64" width="0.1524" layer="91"/>
+<pinref part="R8" gate="G$1" pin="2"/>
+<wire x1="165.1" y1="185.42" x2="167.64" y2="185.42" width="0.1524" layer="91"/>
+<junction x="167.64" y="185.42"/>
+</segment>
+</net>
