File: Eagle/DSP.brd (EAGLE design)
At the start: 100 x 100 mm, 20 parts

Commit message: continuing layout
Parts:
- added C6: 0.1uF, kiss_z:0603
- added R6, R7: 100K, kiss_z:0603
- R1: value 4611X-101-102LF -> 4711X_RES
- moved R5 215.1 mm to (90.8, 50.8), turned to 180 degrees
- moved S2 208.7 mm to (97.2, 55.9), turned to 270 degrees
- moved J4 151.9 mm to (64.8, 41.9), turned to 180 degrees
- moved R4 150.0 mm to (11.4, 50.8), turned to 180 degrees
- moved C4 150.0 mm to (58.4, 6.35)
- moved J1 146.8 mm to (52.1, 6.35), turned to 90 degrees
- moved D1 146.7 mm to (82.5, 8.89), turned to 90 degrees
- moved R1 139.3 mm to (87.6, 6.35), turned to 270 degrees
- moved J3 136.6 mm to (44.5, 36.8), turned to 270 degrees
- moved J2 135.4 mm to (56.5, 50.2)
- moved J5 135.3 mm to (48.3, 66.0)
- moved C3 133.0 mm to (57.8, 52.7), turned to 180 degrees
- moved TEENSY_3.2 131.4 mm to (69.8, 6.35), turned to 180 degrees
- moved S1 116.4 mm to (5.08, 45.7), turned to 90 degrees
- moved C5 110.1 mm to (22.2, 53.3)
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Connections:
- net +3V3: now also C6.1, R6.2
- net GND: now also R7.1
- net N$2: now also R6.1, R7.2
Other:
- board size 100 x 100 mm -> 100 x 75 mm

Commit message: finished DSP layout!
Parts:
- moved R1 78.8 mm to (8.89, 10.2), turned to 180 degrees
- moved C5 55.1 mm to (67.3, 21.6), turned to 90 degrees
- moved R3 54.3 mm to (31.8, 15.2), turned to 270 degrees
- moved J5 53.4 mm to (25.4, 17.8), turned to 180 degrees
- moved C2 50.6 mm to (29.2, 17.8), turned to 0 degrees
- moved R2 44.4 mm to (31.8, 20.3), turned to 270 degrees
- moved D1 43.6 mm to (39.4, 2.54), turned to 0 degrees
- moved TEENSY_3.2 34.2 mm to (36.8, 15.2), turned to 90 degrees
- moved J1 30.7 mm to (36.8, 33.0), turned to 0 degrees
- moved C4 29.6 mm to (38.1, 27.9)
- moved C3 29.4 mm to (73.7, 27.9), turned to 0 degrees
- moved J2 27.0 mm to (74.9, 30.5), turned to 180 degrees
- moved C1 24.0 mm to (24.8, 71.1), turned to 0 degrees
- moved C6 23.6 mm to (79.4, 71.1), turned to 180 degrees
- moved J3 23.2 mm to (67.3, 40.6), turned to 180 degrees
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Connections:
- net +3V3: now also J3.5; no longer J3.3
- net GND: now also C6.2
- net MISO: now also J3.1; no longer J3.2
- net MOSI: now also J3.2; no longer J3.1
- net SCLK: now also J3.3; no longer J3.5
Routing:
- net +3V3: track 0.00 -> 233.6 mm, vias 0 -> 1
- net MOSI: track 0.00 -> 93.5 mm
- net CS_LCD: track 0.00 -> 91.4 mm
- net SCLK: track 0.00 -> 69.6 mm
- net SW_MOM: track 0.00 -> 66.5 mm, vias 0 -> 2
- net RST_LCD: track 0.00 -> 63.2 mm, vias 0 -> 2
- net REG_LCD: track 0.00 -> 62.6 mm, vias 0 -> 2
- net ADC_IN: track 0.00 -> 52.4 mm
- net SW_TOG: track 0.00 -> 45.2 mm
- net MISO: track 0.00 -> 35.7 mm
- net N$6: track 0.00 -> 31.1 mm
- net N$5: track 0.00 -> 31.1 mm
- net N$9: track 0.00 -> 31.1 mm
- net N$8: track 0.00 -> 31.1 mm
- net N$7: track 0.00 -> 31.1 mm
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- added copper zone on layer 16, net GND

Commit message: w00f
Parts:
- added C7: 0.22uF, kiss_z:0603
- added R8: 1K, kiss_z:0603
- moved S2 1.60 mm to (94.9, 55.9)
- moved R6 1.27 mm to (88.9, 54.6)
- moved R7 1.27 mm to (88.9, 47.0)
- moved R5 0.25 mm to (88.0, 50.8)
Connections:
- new net N$24: C7.1, R2.1, R8.2
- net +3V3: now also R8.1; no longer R2.1
- net GND: now also C7.2
Routing:
- net +3V3: track 233.6 -> 225.1 mm
- net N$24: track 0.00 -> 5.07 mm
- net N$2: track 13.5 -> 9.49 mm
- net GND: track 17.0 -> 19.9 mm, vias 2 -> 3
Other:
- board text added: "+3V3"
- board text added: "16"
- board text added: "17"
- board text added: "18"
- board text added: "19"
- board text added: "20"
- board text added: "21"
- board text added: "GND"
- board text added: "KISS RADARS INC DSP R0 Z. DARPINIAN"
- board text added: "MISO"
- board text added: "MOSI"
- board text added: "SCLK"
- board text added: "VIN"

Commit message: fixed trace
Routing:
- net CS_LCD: track 91.4 -> 92.8 mm
Changed lines of the file:
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@@
 <contactref element="U$1" pad="6"/>
 <wire x1="64.77" y1="15.24" x2="66.04" y2="13.97" width="0.4064" layer="1"/>
-<wire x1="78.2574" y1="21.63581875" x2="78.2574" y2="31.70418125" width="0.4064" layer="1"/>
-<wire x1="78.2574" y1="31.70418125" x2="76.15418125" y2="33.8074" width="0.4064" layer="1"/>
-<wire x1="76.15418125" y1="33.8074" x2="76.0476" y2="33.8074" width="0.4064" layer="1"/>
 <wire x1="70.59158125" y1="13.97" x2="78.2574" y2="21.63581875" width="0.4064" layer="1"/>
 <wire x1="66.04" y1="13.97" x2="70.59158125" y2="13.97" width="0.4064" layer="1"/>
-<wire x1="76.0476" y1="33.8074" x2="59.7888" y2="50.0662" width="0.4064" layer="1"/>
 <wire x1="46.68605" y1="50.0662" x2="31.115" y2="65.63725" width="0.4064" layer="1"/>
 <wire x1="31.115" y1="65.63725" x2="31.115" y2="68.58" width="0.4064" layer="1"/>
-<wire x1="59.7888" y1="50.0662" x2="46.68605" y2="50.0662" width="0.4064" layer="1"/>
+<wire x1="78.2574" y1="21.63581875" x2="78.2574" y2="34.1376" width="0.4064" layer="1"/>
+<wire x1="78.2574" y1="34.1376" x2="62.3288" y2="50.0662" width="0.4064" layer="1"/>
+<wire x1="62.3288" y1="50.0662" x2="46.68605" y2="50.0662" width="0.4064" layer="1"/>
 </signal>
 <signal name="MOSI">
