File: Eagle/DSP_DC_SYNTH.sch (EAGLE design)
At the start: 81 parts, among them J2 3.5HEADPHONEJACK, J5 U.FL_CONN, J6 U.FL_CONN, U1 5V_REG, U2 MIXER, U3 DUAL_OP_AMP_LMV822, U4 DIGITAL_POTDIGITAL_POT, U5 TC1185-3.3VCT713, U6 LMX2326, U7 MAX2752, U8 RMK-3-93+

Commit message: updates to combined schem
Parts:
- added J15: (no value), SparkFun-Connectors:CONN_03
- added J16: U.FL_CONN, 764Library:U.FL_CONN
Connections:
- removed net CS_PLL: J13.7, TEENSY_3.2.17
- removed net OSC_EN: J14.2, R21.2, U7.!SHDN, XO1.EN
- removed net PLL_CE: U6.CE
- removed net PLL_CLK: U6.CLOCK
- removed net PLL_MOSI: U6.DATA
- removed net PLL_MUX: J14.7, U6.FO/LD
- new net EXT_REF: J15.3, J16.SIG
- new net OSC_PLL_BU_EN: J14.2, R21.2, TEENSY_3.2.19, U6.CE, U7.!SHDN, XO1.EN
- new net PLL_BU_MUX: J14.7, TEENSY_3.2.18, U6.FO/LD
- new net PLL_IN: C26.2, J15.2
- net 19: no longer TEENSY_3.2.19
- net 20: no longer TEENSY_3.2.20
- net ADC_IN: now also TEENSY_3.2.20; no longer TEENSY_3.2.18
- net FL_OUT: no longer U6.FLO
- net GND: now also J16.GND
- net MOSI: now also U6.DATA
- net PLL_LE: now also J13.7, TEENSY_3.2.17
- net SCLK: now also U6.CLOCK
- net TCXO_OUT: now also J15.1; no longer C26.2
Other:
- note added: "UPDATE VALUES"
- note added: "delete this"
- moved on the sheet: C21, C22, C26, C31, U6, U8

Commit message: more additions
Parts:
- added J17: U.FL_CONN, 764Library:U.FL_CONN
Connections:
- net GND: now also J17.GND
Other:
- note added: "ADD AMPLIFIER"
- note added: "ADD SPLITTER"
Changed lines of the file:
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@@
 <part name="J16" library="764Library" deviceset="U.FL_CONN" device=""/>
 <part name="GND32" library="supply1" library_urn="urn:adsk.eagle:library:371" deviceset="GND" device=""/>
+<part name="J17" library="764Library" deviceset="U.FL_CONN" device=""/>
+<part name="GND33" library="supply1" library_urn="urn:adsk.eagle:library:371" deviceset="GND" device=""/>
 </parts>
 <sheets>
@@
 <plain>
 <text x="228.6" y="30.48" size="1.778" layer="91">Cin = 1/(2*pi*Fin*1Ohm)</text>
-<text x="292.1" y="30.48" size="1.778" layer="91">Cout = 1/(2*pi*Fout*1Ohm)</text>
+<text x="292.1" y="48.26" size="1.778" layer="91">Cout = 1/(2*pi*Fout*1Ohm)</text>
 <text x="15.24" y="53.34" size="1.778" layer="91">Loop Filter</text>
 <text x="228.6" y="50.8" size="1.778" layer="91">X3 Frequency Multiplier</text>
@@
 <text x="53.34" y="165.1" size="3.302" layer="91">delete this</text>
 <text x="40.64" y="53.34" size="3.302" layer="91">UPDATE VALUES</text>
+<text x="172.72" y="53.34" size="3.302" layer="91">ADD AMPLIFIER</text>
+<text x="172.72" y="48.26" size="3.302" layer="91">ADD SPLITTER</text>
+<text x="172.72" y="43.18" size="3.302" layer="91">ADD AMPLIFIER</text>
 </plain>
 <instances>
@@
 </instance>
 <instance part="GND32" gate="1" x="116.84" y="86.36"/>
+<instance part="J17" gate="G$1" x="317.5" y="35.56" smashed="yes" rot="MR0">
+<attribute name="NAME" x="321.31" y="39.624" size="1.778" layer="95" rot="MR0"/>
+<attribute name="VALUE" x="336.804" y="36.322" size="1.778" layer="96" rot="MR0"/>
+</instance>
+<instance part="GND33" gate="1" x="309.88" y="27.94"/>
 </instances>
 <busses>
@@
 <wire x1="116.84" y1="91.44" x2="116.84" y2="88.9" width="0.1524" layer="91"/>
 </segment>
+<segment>
+<pinref part="J17" gate="G$1" pin="GND"/>
+<wire x1="314.96" y1="33.02" x2="309.88" y2="33.02" width="0.1524" layer="91"/>
+<pinref part="GND33" gate="1" pin="GND"/>
+<wire x1="309.88" y1="33.02" x2="309.88" y2="30.48" width="0.1524" layer="91"/>
+</segment>
 </net>
 <net name="CPOUT" class="0">
@@
 <segment>
 <pinref part="C22" gate="G$1" pin="2"/>
-<wire x1="302.26" y1="38.1" x2="304.8" y2="38.1" width="0.1524" layer="91"/>
-<label x="304.8" y="38.1" size="1.778" layer="95"/>
-</segment>
-</net>
+<wire x1="302.26" y1="38.1" x2="314.96" y2="38.1" width="0.1524" layer="91"/>
+</segment>
+</net>
