File: Eagle/DSP_DC_SYNTH.brd (EAGLE design)
At the start: 160 x 100 mm, 83 parts, among them J16 U.FL_CONN, J17 U.FL_CONN, J2 3.5HEADPHONEJACK, J5 U.FL_CONN, J6 U.FL_CONN, U1 5V_REG, U2 MIXER, U3 DUAL_OP_AMP_LMV822, U4 DIGITAL_POTDIGITAL_POT, U5 TC1185-3.3VCT713, U6 LMX2326, U7 MAX2752, U8 RMK-3-93+

Commit message: Updated net names to match for zack's convention
Connections:
- removed net CPOUT: U6.2
- removed net CS: U4.1
- removed net SCK: U4.2
- removed net SDI: U4.3
- removed net SDO: U4.13
- removed net SHDN: U4.12
- new net PLL_CLK: J14.4
- new net PLL_MOSI: J14.5
- net CP_OUT: now also U6.2
- net CS_POT: now also U4.1
- net MISO: now also U4.13
- net MOSI: now also U4.3
- net OSC_PLL_BU_EN: now also J14.3
- net PLL_LE: now also J14.6
- net SCLK: now also U4.2
Changed lines of the file:
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@@
 <wire x1="-100.4062" y1="95.885" x2="-72.81" y2="124.46" width="0" layer="19" extent="1-1"/>
-</signal>
-<signal name="CS">
-<contactref element="U4" pad="1"/>
-</signal>
-<signal name="SCK">
-<contactref element="U4" pad="2"/>
-</signal>
-<signal name="SDI">
-<contactref element="U4" pad="3"/>
 </signal>
 <signal name="AUDIO_OUT">
@@
 <wire x1="-22.5287" y1="97.11" x2="-16.09" y2="129.54" width="0" layer="19" extent="1-1"/>
 <wire x1="-100.4062" y1="97.155" x2="-22.5287" y2="97.11" width="0" layer="19" extent="1-1"/>
-</signal>
-<signal name="SDO">
-<contactref element="U4" pad="13"/>
-</signal>
-<signal name="SHDN">
-<contactref element="U4" pad="12"/>
 </signal>
 <signal name="3.3V">
@@
 <contactref element="J13" pad="2"/>
 <contactref element="U6" pad="12"/>
-<wire x1="-53.34" y1="129.54" x2="-14.9352" y2="107.625" width="0" layer="19" extent="1-1"/>
-<wire x1="-29.21" y1="62.23" x2="-14.9352" y2="107.625" width="0" layer="19" extent="1-1"/>
+<contactref element="U4" pad="3"/>
+<wire x1="-28.2713" y1="99.71" x2="-14.9352" y2="107.625" width="0" layer="19" extent="1-1"/>
+<wire x1="-29.21" y1="62.23" x2="-28.2713" y2="99.71" width="0" layer="19" extent="1-1"/>
+<wire x1="-53.34" y1="129.54" x2="-28.2713" y2="99.71" width="0" layer="19" extent="1-1"/>
 <wire x1="-83.82" y1="2.54" x2="-29.21" y2="62.23" width="0" layer="19" extent="1-1"/>
 </signal>
@@
 <contactref element="TEENSY_3.2" pad="12"/>
 <contactref element="J13" pad="1"/>
-<wire x1="-29.21" y1="59.69" x2="-55.88" y2="129.54" width="0" layer="19" extent="1-1"/>
+<contactref element="U4" pad="13"/>
+<wire x1="-29.21" y1="59.69" x2="-22.5287" y2="100.36" width="0" layer="19" extent="1-1"/>
+<wire x1="-55.88" y1="129.54" x2="-22.5287" y2="100.36" width="0" layer="19" extent="1-1"/>
 </signal>
 <signal name="RST_LCD">
@@
 <contactref element="J13" pad="3"/>
 <contactref element="U6" pad="11"/>
-<wire x1="-50.8" y1="129.54" x2="-14.9352" y2="106.975" width="0" layer="19" extent="1-1"/>
-<wire x1="-13.97" y1="59.69" x2="-14.9352" y2="106.975" width="0" layer="19" extent="1-1"/>
+<contactref element="U4" pad="2"/>
+<wire x1="-28.2713" y1="100.36" x2="-14.9352" y2="106.975" width="0" layer="19" extent="1-1"/>
+<wire x1="-50.8" y1="129.54" x2="-28.2713" y2="100.36" width="0" layer="19" extent="1-1"/>
+<wire x1="-13.97" y1="59.69" x2="-28.2713" y2="100.36" width="0" layer="19" extent="1-1"/>
 <wire x1="-86.36" y1="2.54" x2="-13.97" y2="59.69" width="0" layer="19" extent="1-1"/>
 </signal>
@@
 <contactref element="TEENSY_3.2" pad="16"/>
 <contactref element="J13" pad="6"/>
-<wire x1="-13.97" y1="67.31" x2="-43.18" y2="129.54" width="0" layer="19" extent="1-1"/>
+<contactref element="U4" pad="1"/>
+<wire x1="-28.2713" y1="101.01" x2="-43.18" y2="129.54" width="0" layer="19" extent="1-1"/>
+<wire x1="-13.97" y1="67.31" x2="-28.2713" y2="101.01" width="0" layer="19" extent="1-1"/>
 </signal>
 <signal name="PLL_LE">
@@
 <contactref element="J13" pad="7"/>
 <contactref element="U6" pad="13"/>
+<contactref element="J14" pad="6"/>
 <wire x1="-40.64" y1="129.54" x2="-14.9352" y2="108.274996875" width="0" layer="19" extent="1-1"/>
+<wire x1="-64.77" y1="129.54" x2="-40.64" y2="129.54" width="0" layer="19" extent="1-1"/>
 <wire x1="-13.97" y1="69.85" x2="-14.9352" y2="108.274996875" width="0" layer="19" extent="1-1"/>
 </signal>
@@
 <contactref element="R21" pad="2"/>
 <contactref element="J14" pad="2"/>
+<contactref element="J14" pad="3"/>
 <wire x1="-24.905" y1="107.505" x2="-14.9352" y2="106.325" width="0" layer="19" extent="1-1"/>
 <wire x1="-13.97" y1="74.93" x2="-14.9352" y2="106.325" width="0" layer="19" extent="1-1"/>
 <wire x1="-67.73" y1="124.46" x2="-24.905" y2="107.505" width="0" layer="19" extent="1-1"/>
-<wire x1="-74.93" y1="129.54" x2="-67.73" y2="124.46" width="0" layer="19" extent="1-1"/>
+<wire x1="-72.39" y1="129.54" x2="-67.73" y2="124.46" width="0" layer="19" extent="1-1"/>
+<wire x1="-74.93" y1="129.54" x2="-72.39" y2="129.54" width="0" layer="19" extent="1-1"/>
 <wire x1="-92.3544" y1="105.705" x2="-74.93" y2="129.54" width="0" layer="19" extent="1-1"/>
 </signal>
@@
 <contactref element="C22" pad="1"/>
 <wire x1="-39.37" y1="102.489" x2="-44.03" y2="124.46" width="0" layer="19" extent="1-1"/>
-</signal>
-<signal name="CPOUT">
-<contactref element="U6" pad="2"/>
 </signal>
 <signal name="VCO_OUT">
@@
 <contactref element="R17" pad="2"/>
 <contactref element="U7" pad="2"/>
+<contactref element="U6" pad="2"/>
+<wire x1="-56.73" y1="124.46" x2="-20.6248" y2="109.575" width="0" layer="19" extent="1-1"/>
 <wire x1="-82.97" y1="124.46" x2="-56.73" y2="124.46" width="0" layer="19" extent="1-1"/>
 <wire x1="-92.3544" y1="107.005" x2="-82.97" y2="124.46" width="0" layer="19" extent="1-1"/>
@@
 <wire x1="-85.345" y1="99.06" x2="-42.33" y2="124.46" width="0" layer="19" extent="1-1"/>
 </signal>
+<signal name="PLL_MOSI">
+<contactref element="J14" pad="5"/>
+</signal>
+<signal name="PLL_CLK">
+<contactref element="J14" pad="4"/>
+</signal>
 </signals>

Commit message: started layout
Parts:
- moved U$1 191.9 mm to (89.5, 58.7), turned to 180 degrees
- moved C7 138.0 mm to (32.4, 94.3), turned to 90 degrees
- moved R4 133.0 mm to (21.6, 89.2), turned to 180 degrees
- moved C4 131.1 mm to (37.5, 90.2), turned to 90 degrees
- moved U3 125.5 mm to (21.9, 84.1)
- moved C8 116.3 mm to (23.5, 94.3)
- moved R10 109.7 mm to (27.6, 82.2), turned to 180 degrees
- moved R5 95.7 mm to (26.7, 88.9), turned to 90 degrees
- moved R9 71.8 mm to (24.4, 79.1), turned to 270 degrees
- moved J2 68.6 mm to (16.5, 88.3), turned to 270 degrees
- moved R8 68.5 mm to (21.6, 77.5)
- moved R7 66.7 mm to (19.7, 75.2)
- moved C13 65.1 mm to (27.0, 79.1), turned to 270 degrees
- moved R6 61.0 mm to (34.6, 94.3), turned to 90 degrees
- moved C5 59.9 mm to (28.9, 88.9), turned to 270 degrees
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Other:
- board size 160 x 100 mm -> 100 x 100 mm
